File: PCB Inductive Coils/Ver3.2/SDR1806.brd (EAGLE design)
At the start: 43.9 x 25.4 mm, 6 parts

Commit message: added scripts and PCB files
Parts:
- removed L2, L3: SDR1806, SDR1806:SDR1806
- removed R2: (no value), rcl:R0603
- moved JP1 26.4 mm to (2.29, 21.6), turned to 0 degrees
- moved R1 22.0 mm to (2.54, 2.79), turned to 180 degrees
Connections:
- removed net N$1: L1.2, L2.1
- removed net N$2: L2.2, L3.1
- net N$3: no longer R2.1
- net N$4: now also L1.2; no longer L3.2, R2.2
Routing:
- net N$4: track 62.1 -> 26.0 mm, vias 1 -> 0
- net N$2: track 30.2 -> 0.00 mm
- net N$1: track 28.9 -> 0.00 mm
- net N$3: track 23.1 -> 26.7 mm
Other:
- board size 43.9 x 25.4 mm -> 14.9 x 25.4 mm
Changed lines of the file:
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@@
 <layer number="23" name="tOrigins" color="15" fill="1" visible="yes" active="yes"/>
 <layer number="24" name="bOrigins" color="15" fill="1" visible="yes" active="yes"/>
-<layer number="25" name="tNames" color="7" fill="1" visible="yes" active="yes"/>
-<layer number="26" name="bNames" color="7" fill="1" visible="yes" active="yes"/>
-<layer number="27" name="tValues" color="7" fill="1" visible="yes" active="yes"/>
-<layer number="28" name="bValues" color="7" fill="1" visible="yes" active="yes"/>
+<layer number="25" name="tNames" color="7" fill="1" visible="no" active="yes"/>
+<layer number="26" name="bNames" color="7" fill="1" visible="no" active="yes"/>
+<layer number="27" name="tValues" color="7" fill="1" visible="no" active="yes"/>
+<layer number="28" name="bValues" color="7" fill="1" visible="no" active="yes"/>
 <layer number="29" name="tStop" color="7" fill="3" visible="no" active="yes"/>
 <layer number="30" name="bStop" color="7" fill="6" visible="no" active="yes"/>
@@
 <board>
 <plain>
-<wire x1="0" y1="0" x2="43.866" y2="0" width="0" layer="20"/>
-<wire x1="43.866" y1="0" x2="43.866" y2="25.39" width="0" layer="20"/>
-<wire x1="43.866" y1="25.39" x2="0" y2="25.39" width="0" layer="20"/>
+<wire x1="0" y1="0" x2="14.91" y2="0" width="0" layer="20"/>
+<wire x1="14.91" y1="0" x2="14.91" y2="25.39" width="0" layer="20"/>
+<wire x1="14.91" y1="25.39" x2="0" y2="25.39" width="0" layer="20"/>
 <wire x1="0" y1="25.39" x2="0" y2="0" width="0" layer="20"/>
 </plain>
@@
 </autorouter>
 <elements>
-<element name="JP1" library="jumper" package="JP1" value="" x="28.702" y="22.098" rot="R90"/>
+<element name="JP1" library="jumper" package="JP1" value="" x="2.286" y="21.59"/>
 <element name="L1" library="SDR1806" package="SDR1806" value="SDR1806" x="7.62" y="11.684" rot="R270"/>
-<element name="L2" library="SDR1806" package="SDR1806" value="SDR1806" x="21.844" y="11.684" rot="R270"/>
-<element name="L3" library="SDR1806" package="SDR1806" value="SDR1806" x="36.83" y="11.684" rot="R270"/>
-<element name="R1" library="rcl" package="R0603" value="" x="13.462" y="21.844" rot="R270"/>
-<element name="R2" library="rcl" package="R0603" value="" x="17.018" y="21.844" rot="R270"/>
+<element name="R1" library="rcl" package="R0603" value="" x="2.54" y="2.794" rot="R180"/>
 </elements>
 <signals>
-<signal name="N$1">
-<contactref element="L1" pad="2"/>
-<contactref element="L2" pad="1"/>
-<wire x1="7.62" y1="2.594" x2="12.5" y2="2.594" width="0.8128" layer="1"/>
-<wire x1="12.5" y1="2.594" x2="14.478" y2="4.572" width="0.8128" layer="1"/>
-<wire x1="21.844" y1="20.774" x2="21.844" y2="14.986" width="0.8128" layer="1"/>
-<wire x1="21.844" y1="14.986" x2="19.812" y2="12.954" width="0.8128" layer="1"/>
-<wire x1="19.812" y1="12.954" x2="16.51" y2="12.954" width="0.8128" layer="1"/>
-<wire x1="16.51" y1="12.954" x2="14.478" y2="10.922" width="0.8128" layer="1"/>
-<wire x1="14.478" y1="10.922" x2="14.478" y2="4.572" width="0.8128" layer="1"/>
-</signal>
-<signal name="N$2">
-<contactref element="L2" pad="2"/>
-<contactref element="L3" pad="1"/>
-<wire x1="21.844" y1="2.594" x2="27.486" y2="2.594" width="0.8128" layer="1"/>
-<wire x1="27.486" y1="2.594" x2="29.464" y2="4.572" width="0.8128" layer="1"/>
-<wire x1="29.464" y1="4.572" x2="29.464" y2="14.986" width="0.8128" layer="1"/>
-<wire x1="29.464" y1="14.986" x2="31.242" y2="16.764" width="0.8128" layer="1"/>
-<wire x1="31.242" y1="16.764" x2="35.56" y2="16.764" width="0.8128" layer="1"/>
-<wire x1="35.56" y1="16.764" x2="36.83" y2="18.034" width="0.8128" layer="1"/>
-<wire x1="36.83" y1="18.034" x2="36.83" y2="20.774" width="0.8128" layer="1"/>
-</signal>
 <signal name="N$3">
 <contactref element="L1" pad="1"/>
 <contactref element="JP1" pad="2"/>
 <contactref element="R1" pad="1"/>
-<contactref element="R2" pad="1"/>
-<wire x1="7.62" y1="20.774" x2="9.598" y2="20.774" width="0.8128" layer="1"/>
-<wire x1="9.598" y1="20.774" x2="11.43" y2="22.606" width="0.8128" layer="1"/>
-<wire x1="11.43" y1="22.606" x2="13.374" y2="22.606" width="0.8128" layer="1"/>
-<wire x1="13.374" y1="22.606" x2="13.462" y2="22.694" width="0.6096" layer="1"/>
-<wire x1="13.462" y1="22.694" x2="17.018" y2="22.694" width="0.8128" layer="1"/>
-<wire x1="17.018" y1="22.694" x2="17.106" y2="22.694" width="0.6096" layer="1"/>
-<wire x1="17.106" y1="22.694" x2="18.796" y2="24.384" width="0.8128" layer="1"/>
-<wire x1="18.796" y1="24.384" x2="26.67" y2="24.384" width="0.8128" layer="1"/>
-<wire x1="26.67" y1="24.384" x2="27.432" y2="23.622" width="0.8128" layer="1"/>
-<wire x1="27.432" y1="23.622" x2="27.432" y2="22.098" width="0.8128" layer="1"/>
+<wire x1="4.572" y1="4.572" x2="4.572" y2="12.446" width="0.8128" layer="1"/>
+<wire x1="4.572" y1="12.446" x2="7.62" y2="15.494" width="0.8128" layer="1"/>
+<wire x1="7.62" y1="15.494" x2="7.62" y2="20.774" width="0.8128" layer="1"/>
+<wire x1="7.62" y1="22.098" x2="7.62" y2="20.774" width="0.8128" layer="1"/>
+<wire x1="3.39" y1="2.794" x2="3.39" y2="3.39" width="0.8128" layer="1"/>
+<wire x1="3.39" y1="3.39" x2="4.572" y2="4.572" width="0.8128" layer="1"/>
+<wire x1="7.62" y1="22.098" x2="5.334" y2="22.098" width="0.8128" layer="1"/>
+<wire x1="5.334" y1="22.098" x2="4.572" y2="22.86" width="0.8128" layer="1"/>
+<wire x1="4.572" y1="22.86" x2="2.286" y2="22.86" width="0.8128" layer="1"/>
 </signal>
 <signal name="N$4">
-<contactref element="L3" pad="2"/>
 <contactref element="JP1" pad="1"/>
 <contactref element="R1" pad="2"/>
-<contactref element="R2" pad="2"/>
-<wire x1="13.462" y1="20.994" x2="17.018" y2="20.994" width="0.8128" layer="1"/>
-<wire x1="29.972" y1="22.098" x2="32.512" y2="22.098" width="0.8128" layer="1"/>
-<wire x1="32.512" y1="22.098" x2="34.544" y2="24.13" width="0.8128" layer="1"/>
-<wire x1="34.544" y1="24.13" x2="39.116" y2="24.13" width="0.8128" layer="1"/>
-<wire x1="39.116" y1="24.13" x2="40.64" y2="22.606" width="0.8128" layer="1"/>
-<wire x1="40.64" y1="22.606" x2="40.64" y2="4.064" width="0.8128" layer="1"/>
-<wire x1="40.64" y1="4.064" x2="39.116" y2="2.54" width="0.8128" layer="1"/>
-<wire x1="39.116" y1="2.54" x2="36.884" y2="2.54" width="0.8128" layer="1"/>
-<wire x1="36.884" y1="2.54" x2="36.83" y2="2.594" width="0.6096" layer="1"/>
-<wire x1="17.018" y1="20.994" x2="17.018" y2="19.304" width="0.8128" layer="1"/>
-<wire x1="17.018" y1="19.304" x2="16.256" y2="18.542" width="0.8128" layer="1"/>
-<wire x1="16.256" y1="18.542" x2="14.224" y2="18.542" width="0.8128" layer="1"/>
-<via x="14.224" y="18.542" extent="1-16" drill="0.6" diameter="1.27" shape="octagon"/>
-<wire x1="14.224" y1="18.542" x2="28.448" y2="18.542" width="0.8128" layer="16"/>
-<wire x1="28.448" y1="18.542" x2="29.972" y2="19.558" width="0.8128" layer="16"/>
-<wire x1="29.972" y1="19.558" x2="29.972" y2="22.098" width="0.8128" layer="16"/>
+<contactref element="L1" pad="2"/>
+<wire x1="2.286" y1="16.764" x2="2.286" y2="20.32" width="0.8128" layer="1"/>
+<wire x1="6.985" y1="1.397" x2="7.112" y2="1.524" width="0.8128" layer="1"/>
+<wire x1="7.112" y1="1.524" x2="7.112" y2="2.086" width="0.8128" layer="1"/>
+<wire x1="7.112" y1="2.086" x2="7.62" y2="2.594" width="0.8128" layer="1"/>
+<wire x1="1.69" y1="2.794" x2="1.69" y2="16.168" width="0.8128" layer="1"/>
+<wire x1="1.69" y1="16.168" x2="2.286" y2="16.764" width="0.8128" layer="1"/>
+<wire x1="1.69" y1="2.794" x2="1.69" y2="1.866" width="0.8128" layer="1"/>
+<wire x1="1.69" y1="1.866" x2="2.54" y2="1.016" width="0.8128" layer="1"/>
+<wire x1="2.54" y1="1.016" x2="6.604" y2="1.016" width="0.8128" layer="1"/>
+<wire x1="6.604" y1="1.016" x2="6.985" y2="1.397" width="0.8128" layer="1"/>
 </signal>
 </signals>
